Commit message: Added the bot and blank script files too

File: washroom_cleaner/urdf/washroom_cleaner.urdf (robot description, URDF)
Before this commit: robot washroom_cleaner, 2 links, 1 joints
Links:
- link base_link: geometry collision mesh filename=package://washroom_cleaner/meshes/base_link_washroom.STL; visual mesh filename=package://washroom_cleaner/meshes/base_link_washroom.STL
- link link_1: geometry collision mesh filename=package://washroom_cleaner/meshes/link_1_washroom.STL; visual mesh filename=package://washroom_cleaner/meshes/link_1_washroom.STL
