Commit message: Updated models

File: washroom_cleaner/urdf/bot.urdf (robot description, URDF)
Before this commit: robot bot, 9 links, 8 joints
Links:
- link base_link: mass 159.895891670044 -> 159.9
- link link_1: mass 5.5662115488017 -> 10.098
- link link_1.1: mass 4.42645971483181 -> 0.276359187044582
- link link_2: mass 0.136953822245057 -> 0
Joints:
- joint joint: origin xyz=-0.095207 -0.09121 0 rpy=-1.5708 0 -3.1416 -> xyz=-0.0952067740222446 -0.0912104700012903 0 rpy=-1.5707963267949 0 -3.14159265358979
- joint joint_1: origin xyz=0.276989631668551 -0.62512893323251 0.499886146604718 rpy=-1.57079632679503 -0.340650425389168 -1.57079632679486 -> xyz=0.27699 -0.62513 0.49989 rpy=-1.5708 -0.34065 -1.5708
- joint joint_1.1: axis 0 0 0 -> 0 1 0; origin xyz=0.0780337614790351 0.210065530525591 0.116454203404544 rpy=0.340650425389168 -1.5707963267949 0 -> xyz=0.078034 0.21007 0.11645 rpy=0.34065 -1.5708 0; type fixed -> continuous
- joint joint_1.2.1-2: axis 0.7221 0.69179 0 -> 0.72209941749505 0.691789296862353 0; origin xyz=0.10218 0 0.03719 rpy=-1.5708 -0.4149 -3.1416 -> xyz=0.102177334598959 0 0.0371895084106796 rpy=-1.5707963267949 -0.414898179979398 -3.14159265358979
- joint joint_2.1: origin xyz=-0.16411 -0.01 0.13706 rpy=0 1.4907 0 -> xyz=-0.164114522451131 -0.01 0.137058948749274 rpy=0 1.49067939023891 0

Commit message: Bot Lands Stable Now

File: washroom_cleaner/urdf/bot.urdf (robot description, URDF)
Before this commit: robot bot, 9 links, 8 joints
Links:
- removed link link_1.1
- link base_link: mass 159.9 -> 159.895891670044
- link link_1: mass 10.098 -> 10.1002792021682
- link link_1.2: mass 0.151435450174544 -> 0.18680699175307
- link link_2: mass 0 -> 0.136953822245057
- link link_2.1: mass 4.88576945217599 -> 4.885769452176
Joints:
- removed joint joint_1.1
- joint joint_1.2: origin xyz=-0.0291697643061083 -0.395389209897103 0.124217159492965 rpy=-1.57079632679613 -1.47134555278158 -2.80094222819939 -> xyz=-0.02917 -0.39539 0.12422 rpy=-1.5708 -1.4713 -2.8009
