Commit message: altered sensor

File: washroom_cleaner/urdf/bot.urdf.xacro (robot description, xacro)
@@ -13,26 +13,26 @@
   <!-- Lidar -->
   <xacro:include filename="$(find washroom_cleaner)/urdf/distance_sensor.urdf.xacro" />
-  <xacro:distance_sensor name="dist_N" parent="base_link" ros_topic="scan" frame_name="base_link" update_rate="40" ray_count="320" min_angle="-5" max_angle="5" min_range="0.05" max_range="1" noise="true">
+  <xacro:distance_sensor name="dist_N" parent="base_link" ros_topic="scan" frame_name="base_link" update_rate="40" ray_count="10" min_angle="-2.5" max_angle="2.5" min_range="0.05" max_range="5" noise="true">
     <origin xyz="0.067877 0.39974 -0.05186" rpy="${M_PI} 0 ${M_PI/2}"/>
   </xacro:distance_sensor>
-  <xacro:distance_sensor name="dist_NW" parent="base_link" ros_topic="scan" frame_name="base_link" update_rate="40" ray_count="320" min_angle="-5" max_angle="5" min_range="0.05" max_range="1" noise="true">
+  <xacro:distance_sensor name="dist_NW" parent="base_link" ros_topic="scan" frame_name="base_link" update_rate="40" ray_count="10" min_angle="-2.5" max_angle="2.5" min_range="0.05" max_range="5" noise="true">
     <origin xyz="0.40623 0.33093 -0.05186" rpy="${M_PI} 0 ${2.4267 - M_PI/2}"/>
   </xacro:distance_sensor>
-  <xacro:distance_sensor name="dist_W" parent="base_link" ros_topic="scan" frame_name="base_link" update_rate="40" ray_count="320" min_angle="-5" max_angle="5" min_range="0.05" max_range="1" noise="true">
+  <xacro:distance_sensor name="dist_W" parent="base_link" ros_topic="scan" frame_name="base_link" update_rate="40" ray_count="10" min_angle="-2.5" max_angle="2.5" min_range="0.05" max_range="5" noise="true">
     <origin xyz="0.48675 -0.00026 -0.05186" rpy="${M_PI} 0 0"/>
   </xacro:distance_sensor>
-  <xacro:distance_sensor name="dist_SW" parent="base_link" ros_topic="scan" frame_name="base_link" update_rate="40" ray_count="320" min_angle="-5" max_angle="5" min_range="0.05" max_range="1" noise="true">
+  <xacro:distance_sensor name="dist_SW" parent="base_link" ros_topic="scan" frame_name="base_link" update_rate="40" ray_count="10" min_angle="-2.5" max_angle="2.5" min_range="0.05" max_range="5" noise="true">
     <origin xyz="-0.253597943806856 0.329767311841684 -0.05186" rpy="${M_PI} 0 ${-2.28564794445059 - M_PI/2}"/>
   </xacro:distance_sensor>
-  <xacro:distance_sensor name="dist_S" parent="base_link" ros_topic="scan" frame_name="base_link" update_rate="40" ray_count="320" min_angle="-5" max_angle="5" min_range="0.05" max_range="1" noise="true">
+  <xacro:distance_sensor name="dist_S" parent="base_link" ros_topic="scan" frame_name="base_link" update_rate="40" ray_count="10" min_angle="-2.5" max_angle="2.5" min_range="0.05" max_range="5" noise="true">
     <origin xyz="-0.31325 -0.00026 -0.05186" rpy="${M_PI} 0 ${M_PI}"/>
   </xacro:distance_sensor>
-  <xacro:distance_sensor name="dist_SE" parent="base_link" ros_topic="scan" frame_name="base_link" update_rate="40" ray_count="320" min_angle="-5" max_angle="5" min_range="0.05" max_range="1" noise="true">
+  <xacro:distance_sensor name="dist_SE" parent="base_link" ros_topic="scan" frame_name="base_link" update_rate="40" ray_count="10" min_angle="-2.5" max_angle="2.5" min_range="0.05" max_range="5" noise="true">
     <origin xyz="-0.253597943806856 -0.330287311841684 -0.05186" rpy="${M_PI} 0 ${-0.855944709139206 - M_PI/2}"/>
   </xacro:distance_sensor>
-  <xacro:distance_sensor name="dist_E" parent="base_link" ros_topic="scan" frame_name="base_link" update_rate="40" ray_count="320" min_angle="-5" max_angle="5" min_range="0.05" max_range="1" noise="true">
+  <xacro:distance_sensor name="dist_E" parent="base_link" ros_topic="scan" frame_name="base_link" update_rate="40" ray_count="10" min_angle="-2.5" max_angle="2.5" min_range="0.05" max_range="5" noise="true">
     <origin xyz="0.0678770423730095 -0.40026 -0.05186" rpy="${M_PI} 0 ${-M_PI/2}"/>
   </xacro:distance_sensor>
-  <xacro:distance_sensor name="dist_NE" parent="base_link" ros_topic="scan" frame_name="base_link" update_rate="40" ray_count="320" min_angle="-5" max_angle="5" min_range="0.05" max_range="1" noise="true">
+  <xacro:distance_sensor name="dist_NE" parent="base_link" ros_topic="scan" frame_name="base_link" update_rate="40" ray_count="10" min_angle="-2.5" max_angle="2.5" min_range="0.05" max_range="5" noise="true">
     <origin xyz="0.40623 -0.33145 -0.05186" rpy="${M_PI} 0 ${0.71485 - M_PI/2}"/>
   </xacro:distance_sensor>

File: washroom_cleaner/urdf/kinect.urdf.xacro (robot description, xacro)
@@ -20,5 +20,5 @@
           <origin xyz="0 0 0" rpy="${M_PI/2} 0 ${M_PI/2}" />
           <geometry>
-            <mesh filename="package://washroom_cleaner/meshes/camera.STL" />
+            <mesh filename="package://washroom_cleaner/meshes/camera_bot.STL" />
           </geometry>
         </visual>
@@ -26,5 +26,5 @@
           <origin xyz="0 0 0" rpy="${M_PI/2} 0 ${M_PI/2}" />
           <geometry>
-            <mesh filename="package://washroom_cleaner/meshes/camera.STL" />
+            <mesh filename="package://washroom_cleaner/meshes/camera_bot.STL" />
           </geometry>
         </collision>
